Commit message: Imported upstream version '0.3.1' of 'upstream'

File: heron_description/urdf/accessories.urdf.xacro (robot description, xacro)
@@ -9,6 +9,6 @@
     heron_base/launch/base.launch
   -->
-  <xacro:macro name="rear_plate" params="type">
-    <link name="rear_plate">
+  <xacro:macro name="rear_plate" params="type suffix_ns">
+    <link name="${suffix_ns}rear_plate">
       <visual>
         <origin xyz="0 0 0" rpy="0 0 0" />
@@ -20,18 +20,21 @@
     </link>
     <joint name="rear_plate_joint" type="fixed">
-      <parent link="base_link" />
-      <child link="rear_plate" />
+      <parent link="${suffix_ns}base_link" />
+      <child link="${suffix_ns}rear_plate" />
       <origin xyz="-0.1915 0.0 0.001" />
     </joint>
+    <gazebo reference="${suffix_ns}rear_plate">
+      <material>Gazebo/DarkGrey</material>
+    </gazebo>
   </xacro:macro>
   <!-- If enabled, generate a Novatel Smart6 payload. -->
   <xacro:include filename="accessories/novatel_smart6.urdf.xacro" />
   <xacro:if value="$(optenv HERON_NAVSAT_SMART6 0)">
-    <novatel_smart6 prefix="$(optenv HERON_NAVSAT_SMART6_MOUNT rear)"/>
+    <novatel_smart6 prefix="$(optenv HERON_NAVSAT_SMART6_MOUNT rear)" suffix_ns="$(arg suffix_ns)"/>
     <joint name="$(optenv HERON_NAVSAT_SMART6_MOUNT rear)_navsat_joint" type="fixed">
     <origin xyz="$(optenv HERON_NAVSAT_SMART6_OFFSET -0.25 0 0.08)"
             rpy="$(optenv HERON_NAVSAT_SMART6_RPY 0 0 0)" />
-      <parent link="base_link" />
-      <child link="$(optenv HERON_NAVSAT_SMART6_MOUNT rear)_navsat" />
+      <parent link="$(arg suffix_ns)base_link" />
+      <child link="$(arg suffix_ns)$(optenv HERON_NAVSAT_SMART6_MOUNT rear)_navsat" />
     </joint>
   </xacro:if>
@@ -40,11 +43,12 @@
   <xacro:if value="$(optenv HERON_LASER 0)">
     <sick_lms1xx_mount prefix="$(optenv HERON_LASER_MOUNT front)"
-                       topic="$(optenv HERON_LASER_TOPIC front/scan)"/>
-    <rear_plate type="lidar" />
+                       topic="$(optenv HERON_LASER_TOPIC front/scan)"
+                       suffix_ns="$(arg suffix_ns)"/>
+    <rear_plate type="lidar" suffix_ns="$(arg suffix_ns)" />
     <joint name="$(optenv HERON_LASER_MOUNT front)_laser_mount_joint" type="fixed">
       <origin xyz="$(optenv HERON_LASER_OFFSET 0.0575 0 0.0115)"
               rpy="$(optenv HERON_LASER_RPY 0 0 0)" />
-      <parent link="rear_plate" />
-      <child link="$(optenv HERON_LASER_MOUNT front)_laser_mount" />
+      <parent link="$(arg suffix_ns)rear_plate" />
+      <child link="$(arg suffix_ns)$(optenv HERON_LASER_MOUNT front)_laser_mount" />
     </joint>
   </xacro:if>
@@ -52,23 +56,23 @@
   <xacro:include filename="accessories/axis_ptz.urdf.xacro" />
   <xacro:if value="$(optenv HERON_AXIS_PTZ 0)">
-    <axis_ptz prefix="$(optenv HERON_AXIS_PTZ_MOUNT axis_ptz)"/>
+    <axis_ptz prefix="$(optenv HERON_AXIS_PTZ_MOUNT axis_ptz)" suffix_ns="$(arg suffix_ns)"/>
     <joint name="$(optenv HERON_AXIS_PTZ_MOUNT axis_ptz)_camera_joint" type="fixed">
     <origin xyz="$(optenv HERON_AXIS_PTZ_OFFSET -0.124 0 0.078)"
             rpy="$(optenv HERON_AXIS_PTZ_RPY 0 0 0)" />
-      <parent link="rear_plate" />
-      <child link="$(optenv HERON_AXIS_PTZ_MOUNT axis_ptz)_camera_link" />
+      <parent link="$(arg suffix_ns)rear_plate" />
+      <child link="$(arg suffix_ns)$(optenv HERON_AXIS_PTZ_MOUNT axis_ptz)_camera_link" />
     </joint>
   </xacro:if>
   <xacro:if value="$(optenv HERON_SONAR 0)">
-    <link name="sonar_$(optenv HERON_SONAR_MOUNT surface)" />
+    <link name="$(arg suffix_ns)sonar_$(optenv HERON_SONAR_MOUNT surface)" />
     <joint name="$(optenv HERON_SONAR_MOUNT rear)_sonar_joint" type="fixed">
     <origin xyz="$(optenv HERON_SONAR_OFFSET 0.0 0 -0.10)"
             rpy="$(optenv HERON_SONAR_RPY 0 0 0)" />
-      <parent link="base_link" />
-      <child link="sonar_$(optenv HERON_SONAR_MOUNT surface)" />
+      <parent link="$(arg suffix_ns)base_link" />
+      <child link="$(arg suffix_ns)sonar_$(optenv HERON_SONAR_MOUNT surface)" />
     </joint>
   </xacro:if>
   <xacro:unless value="$(optenv HERON_LASER 0)">
-    <rear_plate type="plain" />
+    <rear_plate type="plain" suffix_ns="$(arg suffix_ns)" />
   </xacro:unless>
 </robot>

File: heron_description/urdf/accessories/axis_ptz.urdf.xacro (robot description, xacro)
@@ -1,6 +1,6 @@
 <?xml version="1.0"?>
 <robot xmlns:xacro="http://www.ros.org/wiki/xacro">
-  <xacro:macro name="axis_ptz" params="prefix">
-  <link name="${prefix}_camera_link">
+  <xacro:macro name="axis_ptz" params="prefix suffix_ns">
+  <link name="${suffix_ns}${prefix}_camera_link">
     <visual>
       <origin xyz="0 0 0" rpy="0 0 0" />

File: heron_description/urdf/accessories/novatel_smart6.urdf.xacro (robot description, xacro)
@@ -1,6 +1,6 @@
 <?xml version="1.0"?>
 <robot xmlns:xacro="http://www.ros.org/wiki/xacro">
-  <xacro:macro name="novatel_smart6" params="prefix">
-  <link name="${prefix}_navsat">
+  <xacro:macro name="novatel_smart6" params="prefix suffix_ns">
+  <link name="${suffix_ns}${prefix}_navsat">
     <visual>
       <origin xyz="0 0 0" rpy="0 0 0" />

File: heron_description/urdf/accessories/sick_lms1xx_mount.urdf.xacro (robot description, xacro)
@@ -2,14 +2,14 @@
 <robot xmlns:xacro="http://www.ros.org/wiki/xacro">
   <xacro:include filename="$(find lms1xx)/urdf/sick_lms1xx.urdf.xacro" />
-  <xacro:macro name="sick_lms1xx_mount" params="prefix topic">
-    <sick_lms1xx frame="${prefix}_laser" topic="${topic}" />
-    <link name="${prefix}_laser_mount"/>
-    <joint name="${prefix}_laser_joint" type="fixed">
+  <xacro:macro name="sick_lms1xx_mount" params="prefix topic suffix_ns">
+    <sick_lms1xx frame="${suffix_ns}${prefix}_laser" topic="${suffix_ns}${topic}" />
+    <link name="${suffix_ns}${prefix}_laser_mount"/>
+    <joint name="${suffix_ns}${prefix}_laser_joint" type="fixed">
       <!-- This offset is from the base of the bracket to the LIDAR's focal point. -->
       <origin xyz="0 0 0.149" rpy="0 0 0" />
-      <parent link="${prefix}_laser_mount" />
-      <child link="${prefix}_laser" />
+      <parent link="${suffix_ns}${prefix}_laser_mount" />
+      <child link="${suffix_ns}${prefix}_laser" />
     </joint>
-    <gazebo reference="${prefix}_laser_mount">
+    <gazebo reference="${suffix_ns}${prefix}_laser_mount">
       <material>Gazebo/DarkGrey</material>
     </gazebo>

File: heron_description/urdf/heron.urdf.xacro (robot description, xacro)
@@ -25,99 +25,38 @@
 This program contains the description of the robot base model for the Clearpath Heron
 -->
-<robot name="heron" xmlns:xacro="http://www.ros.org/wiki/xacro">
-    <xacro:property name="PI" value="3.1415926535897931" />
-    <xacro:property name="dummy_inertia" value="1e-09"/>
-    <material name="black"><color rgba="0.0 0.0 0.0 1.0"/></material>
-    <material name="gray"><color rgba="0.7 0.7 0.7 1.0"/></material>
-    <material name="dark_gray"><color rgba="0.2 0.2 0.2 1.0"/></material>
-    <material name="white"><color rgba="1.0 1.0 1.0 1.0"/></material>
-    <material name="yellow"><color rgba="0.8 0.8 0.0 1.0"/></material>
-    <xacro:macro name="panel" params="side location">
-      <!-- location flips the panel. 1 is for the left and -1 is for the right -->
-      <joint name="base_${side}_joint" type="fixed">
-        <origin xyz="0.0 ${location*0.34495} 0.04959" rpy="0 0 0" />
-        <parent link="base_link" />
-        <child link="${side}_panel_link" />
-      </joint>
-      <link name="${side}_panel_link">
-        <inertial>
-          <mass value="0.1" />
-          <origin xyz="0.00000000 0.00000000 0.00000000" />
-          <inertia ixx="0.01" ixy="0.00" ixz="0.00"
-            iyy="0.01" iyz="0.00" izz="0.01" />
-        </inertial>
-        <visual>
-          <origin xyz="0 0 0" rpy="0 0 0" />
-          <geometry>
-            <mesh filename="package://heron_description/meshes/${side}_panel.stl" />
-          </geometry>
-          <material name="yellow" />
-        </visual>
-        <collision>
-          <origin xyz="0 0 0" rpy="0 0 0"/>
-          <geometry>
-            <!-- The collision boundary for parts are taken into account by collision boundary of the base_link. -->
-            <box size="0.001 0.001 0.001" />
-          </geometry>
-        </collision>
-      </link>
-    </xacro:macro>
-    <link name="base_link">
-        <inertial>
-          <mass value="29" />
-          <!-- This is the pose of the inertial reference frame, relative to the link reference frame.
-               The origin of the inertial reference frame needs to be at the center of gravity.
-               The axes of the inertial reference frame do not need to be aligned with the
-               principal axes of the inertia. -->
-          <origin xyz="0 0 0" />
-          <!-- The 3x3 rotational inertia matrix. Because the rotational inertia matrix is symmetric,
-               only 6 above-diagonal elements of this matrix are specified here, using the attributes
-              ixx, ixy, ixz, iyy, iyz, izz.-->
-          <inertia ixx="10" ixy="0" ixz="0" iyy="10" iyz="0" izz="10" />
-        </inertial>
-        <visual>
-          <origin xyz="0 0 0" rpy="0 0 0" />
-          <geometry>
-            <mesh filename="package://heron_description/meshes/heron_base.stl" />
-          </geometry>
-          <material name="dark_gray" />
-        </visual>
-        <collision>
-          <origin xyz="0 0 0" rpy="0 0 0" />
-          <geometry>
-            <box size = "0.1 0.1 0.1"/> <!--making it slightly bigger in x and z direction-->
-          </geometry>
-        </collision>
-    </link>
-    <!-- Side Panels -->
-    <panel side="left" location="1" />
-    <panel side="right" location="-1" />
-    <link name="imu_link">
-      <inertial>
-        <mass value="0.001"/>
-        <origin xyz="0 0 0" rpy="0 0 0"/>
-        <inertia ixx="${dummy_inertia}" ixy="0.0" ixz="0.0" iyy="${dummy_inertia}" iyz="0.0" izz="${dummy_inertia}"/>
-      </inertial>
-    </link>
-    <joint name="imu_joint" type="fixed">
-      <parent link="base_link" />
-      <child link="imu_link" />
-      <origin xyz="$(optenv HERON_IMU_UM6_XYZ -0.290 0.0 0.024)"
-              rpy="$(optenv HERON_IMU_UM6_RPY 3.14159 0.0 0.0)" />
-    </joint>
-    <link name="navsat_link" />
-    <joint name="navsat_joint" type="fixed">
-      <parent link="base_link" />
-      <child link="navsat_link" />
-      <origin xyz="$(optenv HERON_NAVSAT_UBLOX_XYZ 0.015 0.050 0.072)"
-              rpy="$(optenv HERON_NAVSAT_UBLOX_RPY 0.0 0.0 0.0)" />
-    </joint>
-    <!-- Bring in simulation data for Gazebo. -->
-    <xacro:include filename="$(find heron_description)/urdf/heron.gazebo" />
-    <!-- Optional standard accessories, including their simulation data. The rendering
-         of these into the final description is controlled by optenv variables, which
-         default each one to off.-->
-    <xacro:include filename="$(find heron_description)/urdf/accessories.urdf.xacro" />
-    <!-- Optional custom includes. -->
-    <xacro:include filename="$(optenv HERON_URDF_EXTRAS empty.urdf)" />
+<robot name="heron" xmlns:xacro="http://www.ros.org/wiki/xacro" >
+  <xacro:arg name="debug" default="0"/>
+  <xacro:arg name="namespace" default=""/>
+  <xacro:arg name="suffix_ns" default="$(arg namespace)"/>
+  <!-- Include the ROV macro file -->
+  <xacro:include filename="$(find heron_description)/urdf/base.xacro"/>
+  <xacro:include filename="$(find heron_description)/urdf/gazebo.xacro"/>
+  <!-- Create the heron -->
+  <xacro:heron_base namespace="$(arg suffix_ns)">
+    <!-- The underwater object plugin is given as an input block parameter to
+     allow the addition of external models of manipulator units -->
+    <gazebo>
+      <plugin name="uuv_plugin" filename="libuuv_underwater_object_ros_plugin.so">
+        <fluid_density>1028.0</fluid_density>
+        <flow_velocity_topic>hydrodynamics/current_velocity</flow_velocity_topic>
+        <debug>$(arg debug)</debug>
+        <!-- Adding the hydrodynamic and hydrostatic parameters for the vehicle-->
+        <xacro:heron_hydro_model namespace="$(arg suffix_ns)" />
+        <!--
+          In case other modules are added to the vehicle (such as a manipulator)
+          that also have link running with the underwater object plugin, they
+          should also be added in this block. For this, this new module should
+          have a file similar to gazebo.xacro above with the description of the
+          parameter necessary for the underwater object plugin to be initialized.
+        -->
+      </plugin>
+    </gazebo>
+  </xacro:heron_base>
+  <!-- Joint state publisher plugin -->
+  <gazebo>
+    <plugin name="joint_state_publisher" filename="libuuv_joint_state_publisher.so">
+      <robotNamespace>/$(arg namespace)</robotNamespace>
+      <updateRate>10</updateRate>
+    </plugin>
+  </gazebo>
 </robot>
